File: Hardware/Top/fitnessBuddy-TOP.sch (EAGLE design)
At the start: 51 parts, among them SW1 SWITCH.MOM, SW2 SWITCH.MOM, U2 NRF52832_MODULE_MDBT42, U4 PCF8523

Commit message: added FTDI controller
Parts:
- removed R8: 10k, LinnesLab-Passives:RESISTOR0603
- added C22: 100n, LinnesLab-Passives:CAPACITOR0603
- added C23, C24: 47p, LinnesLab-Passives:CAPACITOR0603
- added JP2: (no value), LinnesLab-Switches:JUMPER-SMT_2_NO_SILK
- added LED5: RED, LinnesLab-LED:LED0603
- added LED6: YELLOW, LinnesLab-LED:LED0603
- added R1, R2: 0, LinnesLab-Passives:RESISTOR0603
- added R10: 10k, LinnesLab-Passives:RESISTOR0603
- added R17, R18: 27, LinnesLab-Passives:RESISTOR0603
- added R19, R20: 1k, LinnesLab-Passives:RESISTOR0603
- added U5: FT231XS, LinnesLab-DigitalIC:FT231XS
Connections:
- removed net RXD: U2.P0.08
- removed net TXD: U2.P0.06
- new net !CTS: JP2.2, U5.!CTS
- new net !DTR: U5.!DTR
- new net FT3V3: U5.3V3OUT
- new net N$23: R17.2, U5.USBDM
- new net N$24: R18.2, U5.USBDP
- new net N$25: LED5.C, R19.2
- new net N$26: LED6.C, R20.2
- new net RXD.FT: R2.1, U5.RXD
- new net RXD.NRF: R1.2, U2.P0.08
- new net RXLED: R19.1, U5.CBUS1
- new net TXD.FT: R1.1, U5.TXD
- new net TXD.NRF: R2.2, U2.P0.06
- new net TXLED: R20.1, U5.CBUS2
- net 3.3V: now also C22.2, LED5.A, LED6.A, R10.2, U5.!RESET, U5.VCCIO; no longer R8.2
- net GND: now also C22.1, C23.2, C24.1, JP2.1, U5.GND@16, U5.GND@6
- net SCL: now also R10.1; no longer R8.1
- net USB+: now also C23.1, R18.1
- net USB-: now also C24.2, R17.1
- net V_USB: now also U5.VCC
Other:
- note added: "FTDI Serial-to-USB-Converter"
- note added: "I don't remember if CTS needs to be grounded or left floating so here's a jumper to ground so it can be configued either way dynamically."
- note added: "Notes"
- note added: "TXD goes to RX on the other device RXD goes to TX on the other device"
- moved on the sheet: C10, C11, C12, C7, C8, C9, L2, LED3, LED4, R3, R4, R9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

Commit message: finished bottom board and schematic
Connections:
- removed net BATT: R13.1, R14.2
- removed net CD1: SD2.CARD_DETECT
- removed net CHRG.STAT: CHRG2.STAT, R12.1
- removed net CS.OLED: U3./CS
- removed net DC.OLED: U3.DC/I2C_SA0
- removed net RESET.OLED: U3./RES
- removed net SD.CS: SD2.CS
- removed net SW1: SW1.1, SW2.1
- new net A4/BATT: R13.1, R14.2, U2.P0.28/AIN4
- new net A6/TIA: U2.P0.30/AIN6
- new net A7/PPG: U2.P0.31/AIN7
- new net D11/SW1: SW1.1, U2.P0.11
- new net D15/SW2: SW2.1, U2.P0.15
- new net D16/CS.OLED: U2.P0.16, U3./CS
- new net D27/CHRG.STATUS: CHRG2.STAT, R12.1, U2.P0.27
- new net D29/LED.CTRL: U2.P0.29/AIN5
- new net D3/RESET.OLED: U2.P0.03/AIN1, U3./RES
- new net D4/DC.OLED: U2.P0.04/AIN2, U3.DC/I2C_SA0
- new net D5/CD1: SD2.CARD_DETECT, U2.P0.05/AIN3
- new net D7/SD.CS: SD2.CS, U2.P0.07
Other:
- note added: "Digital Output"

Commit message: Made progress on routing bottom board
Parts:
- removed C2, C5, C6: 1u, LinnesLab-Passives:CAPACITOR0603
- removed C20, C21: 4.7u, LinnesLab-Passives:CAPACITOR0603
- removed CHRG2: MCP73831, LinnesLab-Power:MCP73831
- removed LDO2: MIC5504, LinnesLab-Power:MIC5504
- removed R11: (no value), LinnesLab-Passives:RESISTOR0603
- removed R12, R15: 100k, LinnesLab-Passives:RESISTOR0603
- removed SD2: (no value), LinnesLab-Connectors:MICROSD
- removed U4: PCF8523, LinnesLab-Clocks:PCF8523
- removed XTAL3: 32.7680kHz, LinnesLab-Clocks:CRYSTALECS-.327-12.5-12-C-TR
Connections:
- removed net CD2: SD2.CARD_DETECT1
- removed net N$17: CHRG2.PROG, R11.2
- removed net N$19: U4.OSCO, XTAL3.1
- removed net N$20: U4.OSCI, XTAL3.2
- removed net VBATT: U4.VBAT
- net 3.3V: no longer C2.1, C6.1, LDO2.OUT, R15.2, SD2.VDD, U4.VDD
- net D27/CHRG.STATUS: no longer CHRG2.STAT, R12.1
- net D5/CD1: no longer SD2.CARD_DETECT
- net D7/SD.CS: no longer SD2.CS
- net GND: no longer C2.2, C20.2, C21.1, C5.1, C6.2, CHRG2.VSS, LDO2.GND, R11.1, R15.1, SD2.GND, SD2.GND1, SD2.VSS, U4.VSS
- net MISO: no longer SD2.DATA_OUT
- net MOSI: no longer SD2.DATA_IN
- net SCK: no longer SD2.SCLK
- net SCL: no longer U4.SCL
- net SDA: no longer U4.SDA
- net VIN: no longer C21.2, C5.2, CHRG2.VIN, LDO2.EN, LDO2.IN, R12.2
- net VLIPO: no longer C20.1, CHRG2.VBAT
Other:
- note removed: "Back-up battery if desired"
- note removed: "Connect MISO, MOSI, and SCK to appropriate pins on microcontroller. Those are SPI pins and are generally prespecified. You have more flexibility with the SD.CS pin."
- note removed: "Digital Output"
- note removed: "I2C Address = 0x68h"
- note removed: "Real-time Clock"
- note removed: "SD Card"

Commit message: Began routing top board
Parts:
- removed C17, C18, C19: 2.2uF, LinnesLab-Passives:CAPACITOR0402
- removed C22: 100n, LinnesLab-Passives:CAPACITOR0603
- removed C23, C24: 47p, LinnesLab-Passives:CAPACITOR0603
- removed D4: (no value), LinnesLab-DiscreteSemi:SCHOTTKY-USC
- removed LED5: RED, LinnesLab-LED:LED0603
- removed LED6: YELLOW, LinnesLab-LED:LED0603
- removed R18: 27, LinnesLab-Passives:RESISTOR0603
- removed R20: 1k, LinnesLab-Passives:RESISTOR0603
- removed U5: FT231XS, LinnesLab-DigitalIC:FT231XS
- added C1: 1u, LinnesLab-Passives:CAPACITOR0603
- added C2: 10u, LinnesLab-Passives:CAPACITOR0805
- added C3, C4: (no value), LinnesLab-Passives:CAPACITOR0603
- added C5, C6: 300p, LinnesLab-Passives:CAPACITOR0603
- added D3: (no value), LinnesLab-DiscreteSemi:SCHOTTKY-USC
- added J1: (no value), LinnesLab-Connectors:CONN_02
- added LED1: RED, LinnesLab-LED:LED0603
- added LED2: BLUE, LinnesLab-LED:LED0603
- added R12: 390k, LinnesLab-Passives:RESISTOR0603
- added R15: 0, LinnesLab-Passives:RESISTOR0603
- added U1: NRF52832_MODULE_MDBT42, LinnesLab-Microcontrollers:NRF52832_MODULE_MDBT42
- C10: value 300p -> 100n
- C11: value 300p -> 10uF
- C12: value 10u -> 2.2uF; device LinnesLab-Passives:CAPACITOR0805 -> LinnesLab-Passives:CAPACITOR0402
- C14: value 100n -> 2.2uF; device LinnesLab-Passives:CAPACITOR0603 -> LinnesLab-Passives:CAPACITOR0402
- C16: value 10uF -> 2.2uF; device LinnesLab-Passives:CAPACITOR0603 -> LinnesLab-Passives:CAPACITOR0402
- C7: value 1u -> 100n
- C8, C9: value (none) -> 47p
- J2: device LinnesLab-Connectors:CONN_02 -> LinnesLab-Connectors:CONN_07-1.27MM
- LED4: value BLUE -> YELLOW
- R1, R2: value 0 -> 10k
- R13: value 100k -> 1k
- R14: value 100k -> 0
- R4: value 1k -> 100k
- R5: value 10k -> 100k
- R6: value 10k -> 1k
- R7: value 390k -> 10k
- R9: value 10k -> 27
- SW1, SW2: value SWITCH.MOM -> (none); device LinnesLab-Switches:SWITCH.MOM -> LinnesLab-Switches:SPST-PTS830GG140-COPY.1-3
- SW3, SW4: value (none) -> SWITCH.MOM; device LinnesLab-Switches:SPST-PTS830GG140-COPY.1-3 -> LinnesLab-Switches:SWITCH.MOM
- U2: value NRF52832_MODULE_MDBT42 -> FT231XS; device LinnesLab-Microcontrollers:NRF52832_MODULE_MDBT42 -> LinnesLab-DigitalIC:FT231XS
- renumbered CORTEX1 to DEBUG1, D5 to D2, JP2 to JP1, L2 to L1, R17 to R8, R19 to R11, USB2 to USB1, XTAL2 to XTAL1
Connections:
- net !CTS: now also U2.!CTS; no longer U5.!CTS
- net !DTR: now also U2.!DTR; no longer U5.!DTR
- net 3.3V: now also C10.2, C15.2, C16.2, C2.2, D3.C, J2.4, LED3.A, LED4.A, R1.2, R2.2, R7.2, U1.VDD, U2.!RESET, U2.VCCIO; no longer C12.2, C17.2, C19.2, C22.2, D1.C, LED5.A, LED6.A, R10.2, R5.2, R9.2, U2.VDD, U5.!RESET, U5.VCCIO
- net A4/BATT: now also R4.1, R5.2, U1.P0.28/AIN4; no longer R13.1, R14.2, U2.P0.28/AIN4
- net A6/TIA: now also J2.6, U1.P0.30/AIN6; no longer U2.P0.30/AIN6
- net A7/PPG: now also J2.7, U1.P0.31/AIN7; no longer U2.P0.31/AIN7
- net D11/SW1: now also SW3.1, U1.P0.11; no longer SW1.1, U2.P0.11
- net D15/SW2: now also SW4.1, U1.P0.15; no longer SW2.1, U2.P0.15
- net D16/CS.OLED: now also U1.P0.16; no longer U2.P0.16
- net D27/CHRG.STATUS: now also U1.P0.27; no longer U2.P0.27
- net D29/LED.CTRL: now also J2.5, U1.P0.29/AIN5; no longer U2.P0.29/AIN5
- net D3/RESET.OLED: now also U1.P0.03/AIN1; no longer U2.P0.03/AIN1
- net D4/DC.OLED: now also U1.P0.04/AIN2; no longer U2.P0.04/AIN2
- net D5/CD1: now also U1.P0.05/AIN3; no longer U2.P0.05/AIN3
- net D7/SD.CS: now also U1.P0.07; no longer U2.P0.07
- net DFU: now also SW1.B, U1.P0.20; no longer SW3.B, U2.P0.20
- net DTR: now also C7.1; no longer C14.1
- net FRST: now also U1.P0.22; no longer U2.P0.22
- net FT3V3: now also U2.3V3OUT; no longer U5.3V3OUT
- net GND: now also C1.2, C10.1, C11.1, C13.1, C15.1, C2.1, C3.1, C4.2, C5.2, C6.2, J1.1, J2.3, LED1.C, LED2.C, R10.1, R12.2, R5.1, SW1.A, SW2.B, SW3.3, SW3.4, SW4.3, SW4.4, U1.GND@1, U1.GND@2, U1.GND@3, U1.GND@4, U2.GND@16, U2.GND@6; no longer C10.2, C11.2, C12.1, C17.1, C18.1, C19.1, C22.1, C23.2, C24.1, C7.2, J2.1, LED3.C, LED4.C, R14.1, R6.1, R7.2, SW1.3, SW1.4, SW2.3, SW2.4, SW3.A, SW4.B, U2.GND@1, U2.GND@2, U2.GND@3, U2.GND@4, U5.GND@16, U5.GND@6
- net LED1: now also U1.P0.17; no longer U2.P0.17
- net LED2: now also R6.2, U1.P0.19; no longer R4.2, U2.P0.19
- net MISO: now also U1.P0.14; no longer U2.P0.14
- net MOSI: now also U1.P0.13; no longer U2.P0.13
- net N$1: now also R10.2; no longer R6.2
- net N$10: now also LED2.A, R6.1; no longer LED4.A, R4.1
- net N$11: now also U1.DCC; no longer U2.DCC
- net N$12: now also C1.1, U1.DEC4; no longer C7.1, U2.DEC4
- net N$13: now also C11.2; no longer C16.2
- net N$15: now also C13.2; no longer C18.2
- net N$2: now also R12.1; no longer R7.1
- net N$23: now also U2.USBDM; no longer U5.USBDM
- net N$24: now also R9.2, U2.USBDP; no longer R18.2, U5.USBDP
- net N$25: now also LED3.C; no longer LED5.C
- net N$26: now also LED4.C, R13.2; no longer LED6.C, R20.2
- net N$3: now also C14.2; no longer C13.2
- net N$4: now also C3.2, U1.P0.00/XL1; no longer C8.2, U2.P0.00/XL1
- net N$5: now also C14.1; no longer C13.1
- net N$6: now also C4.1, U1.P0.01/XL2; no longer C9.1, U2.P0.01/XL2
- net N$7: now also C12.2; no longer C15.2
- net N$8: now also C12.1; no longer C15.1
- net N$9: now also LED1.A; no longer LED3.A
- net P0.09/NFC1: now also C5.1, U1.P0.09; no longer C11.1, U2.P0.09
- net P0.10/NFC2: now also C6.1, U1.P0.10; no longer C10.1, U2.P0.10
- net RESET: now also C7.2, D3.A, R7.1, SW2.A, U1.P0.21/RESET; no longer C14.2, D1.A, R5.1, SW4.A, U2.P0.21/RESET
- net RXD.FT: now also R15.1, U2.RXD; no longer R2.1, U5.RXD
- net RXD.NRF: now also R14.2, U1.P0.08; no longer R1.2, U2.P0.08
- net RXLED: now also U2.CBUS1; no longer U5.CBUS1
- net SCK: now also U1.P0.12; no longer U2.P0.12
- net SCL: now also J2.2, R2.1, U1.P0.26; no longer R10.1, U2.P0.26
- net SDA: now also J2.1, R1.1, U1.P0.25; no longer R9.1, U2.P0.25
- net SWCLK: now also U1.SWDCLK; no longer U2.SWDCLK
- net SWDIO: now also U1.SWDIO; no longer U2.SWDIO
- net SWO: now also U1.P0.18/SWO; no longer U2.P0.18/SWO
- net TXD.FT: now also R14.1, U2.TXD; no longer R1.1, U5.TXD
- net TXD.NRF: now also R15.2, U1.P0.06; no longer R2.2, U2.P0.06
- net TXLED: now also R13.1, U2.CBUS2; no longer R20.1, U5.CBUS2
- net USB+: now also C9.1, R9.1; no longer C23.1, R18.1
- net USB-: now also C8.2; no longer C24.2
- net VIN: now also D1.C; no longer D4.C
- net VLIPO: now also D1.A, J1.2, R4.2; no longer D4.A, J2.2, R13.2
- net V_USB: now also U2.VCC; no longer U5.VCC
Other:
- note added: "Connection to bottom board"
- moved on the sheet: C10, C11, C12, C13, C14, C15, C16, C7, C8, C9, D1, LED3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
